Commit message: updated apriltag stuff

File: AuE893_Catkin_WS/src/auefinals/turtlebot3_burger.gazebo.xacro (robot description, xacro)
@@ -124,3 +124,12 @@
     </sensor>
   </gazebo>
+   <gazebo reference="april_tag_link">
+    <mu1>0.1</mu1>
+    <mu2>0.1</mu2>
+    <kp>1000000.0</kp>
+    <kd>100.0</kd>
+    <minDepth>0.001</minDepth>
+    <maxVel>1.0</maxVel>
+    <material>april_tag</material>
+  </gazebo>
 </robot>
